File: PCB/Eagle/Resistor Board/Resistor Board.brd (EAGLE design)
At the start: 65.7 x 63.5 mm, 25 parts

Commit message: Add files via upload
Other:
- board size 65.7 x 63.5 mm -> 68.2 x 67.3 mm
- board text added: "UFSJ / LINNce"
