File: PCB/Eagle/Resistor Board/Resistor Board.sch (EAGLE design)
At the start: 25 parts

Commit message: Add files via upload
Changed lines of the file:
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@@
+</segment>
+</net>
+<net name="N$25" class="0">
+<segment>
+<wire x1="12.7" y1="58.42" x2="60.96" y2="58.42" width="0.1524" layer="91"/>
+<wire x1="60.96" y1="58.42" x2="60.96" y2="73.66" width="0.1524" layer="91"/>
+<wire x1="60.96" y1="73.66" x2="10.16" y2="73.66" width="0.1524" layer="91"/>
+<wire x1="10.16" y1="73.66" x2="10.16" y2="58.42" width="0.1524" layer="91"/>
+<wire x1="10.16" y1="58.42" x2="12.7" y2="58.42" width="0.1524" layer="91"/>
 </segment>
 </net>
